File: Data_Station_All_In_One.sch (KiCad schematic (older format))
At the start: 55 parts, among them J1 Conn_01x02_Male, J10 Conn_01x02_Male, J11 USB_B_Micro, J12 Conn_01x02_Male, J2 Conn_01x02_Male, J3 Conn_01x02_Male, J4 Conn_01x02_Male, J5 Conn_01x02_Male, J6 Conn_01x02_Male, J7 Conn_01x06_Male, J8 Conn_01x06_Male, J9 Conn_01x03_Male, Q1 2N2222, Q2 2N2222, U1 LM7805_TO220, U2 ATMEGA328P-PU, U3 FT232RL, Y1 Crystal

Commit message: updated to reflect actual order
Parts:
- U2: symbol Data_Station_All_In_One-rescue:ATMEGA328P-PU-atmel -> Data_Station_All_In_One-rescue:ATMEGA328P-PU-atmel-Data_Station_All_In_One-rescue
- U3: symbol Data_Station_All_In_One-rescue:FT232RL-Interface_USB -> Data_Station_All_In_One-rescue:FT232RL-Interface_USB-Data_Station_All_In_One-rescue
Changed lines of the file:
@@
 Connection ~ 1500 5100
 $Comp
-L Data_Station_All_In_One-rescue:ATMEGA328P-PU-atmel U2
+L Data_Station_All_In_One-rescue:ATMEGA328P-PU-atmel-Data_Station_All_In_One-rescue U2
 U 1 1 5DFB62E0
 P 2500 3900
@@
 Connection ~ 1200 2800
 $Comp
-L Data_Station_All_In_One-rescue:FT232RL-Interface_USB U3
+L Data_Station_All_In_One-rescue:FT232RL-Interface_USB-Data_Station_All_In_One-rescue U3
 U 1 1 5E0975E0
 P 6500 5050
